File: src/electronics/3DBoard/3DBoard.sch (EAGLE design)
At the start: 30 parts, among them IC1 78L05Z, IC10 2987-DRV8825, IC2 2987-DRV8825, IC3 2987-DRV8825, IC4 2987-DRV8825, IC5 2987-DRV8825, IC6 2987-DRV8825, IC7 2987-DRV8825, IC8 2987-DRV8825, IC9 2987-DRV8825

Commit message: Wiring added and schematics are cleaner.
Parts:
- removed U$1: ESP32DEVKITV1, ESP32-DEVKITV1:ESP32DEVKITV1
- added IC11: 74S139N, 74xx-us:74S139N
- added R10, R2, R3, R4, R5, R6, R7, R8, R9: 10k, rcl:R-US_0204/7
- added U$3, U$4, U$5: CMX60D10, CMX60D10:CMX60D10
- added U1: ESP32-DEVKIT-V1, ESP32-DEVKIT-V1:ESP32-DEVKIT-V1
Connections:
- removed net N$34 (its old number): F1.2, IC1.VI, IC10.VMOT, IC2.VMOT, IC3.VMOT, IC4.VMOT, IC5.VMOT, IC6.VMOT, IC7.VMOT, IC8.VMOT, IC9.VMOT, U$1.VIN
- removed net N$35 (its old number): C1.-, IC1.GND, IC10.GND2, IC2.GND2, IC3.GND2, IC4.GND2, IC5.GND2, IC7.GND2, IC8.GND2, IC9.GND2, SL1.1, SL2.1, SV10.2, SV11.2, SV12.2, U$1.GND1, U$2.GND
- removed net N$47 (its old number): F1.1, SL1.2
- removed net N$48: C1.+, R1.1, SL2.2
- new net N$2: IC10.VMOT, U$5.+DCLOAD
- new net N$3: IC6.VMOT, IC7.VMOT, IC8.VMOT, IC9.VMOT, U$4.+DCLOAD
- new net N$4: IC2.VMOT, IC3.VMOT, IC4.VMOT, IC5.VMOT, U$3.+DCLOAD
- new net N$46: F1.1, SL1.1
- new net N$53: IC3.DIR, U1.D5
- new net N$54: IC3.STEP, U1.D12
- new net N$55: IC4.DIR, U1.D13
- new net N$56: IC4.STEP, U1.D14
- new net N$57: IC5.DIR, U1.D15
- new net N$58: IC2.!RST, IC2.!SLP
- new net N$59: IC3.!RST, IC3.!SLP
- new net N$6: IC2.STEP, U1.D4
- new net N$60: IC4.!RST, IC4.!SLP
- new net N$61: IC5.!RST, IC5.!SLP
- new net N$62: IC6.!RST, IC6.!SLP
- new net N$63: IC7.!RST, IC7.!SLP
- new net N$64: IC8.!RST, IC8.!SLP
- new net N$65: IC9.!RST, IC9.!SLP
- new net N$66: IC10.!RST, IC10.!SLP
- new net N$67: IC2.!EN, R2.2
- new net N$68: IC3.!EN, R3.2
- new net N$69: IC4.!EN, R4.2
- new net N$70: IC5.!EN, R5.2
- new net N$71: IC7.!EN, R6.2
- new net N$72: IC8.!EN, R7.2
- new net N$73: IC9.!EN, R8.2
- new net N$74: IC10.!EN, R9.2
- new net N$75: IC6.!EN, R10.2
- new net N$76: IC5.STEP, U1.D18
- new net N$77: IC6.DIR, U1.D19
- new net N$78: F1.2, IC1.VI, U$3.-DCLOAD, U$4.-DCLOAD, U$5.-DCLOAD, U1.VIN
- new net N$79: IC1.VO, IC10.M0, IC10.M1, IC10.M2, IC2.M0, IC2.M1, IC2.M2, IC3.M0, IC3.M1, IC3.M2, IC4.M0, IC4.M1, IC4.M2, IC5.M0, IC5.M1, IC5.M2, IC6.M0, IC6.M1, IC6.M2, IC7.M0, IC7.M1, IC7.M2, IC8.M0, IC8.M1, IC8.M2, IC9.M0, IC9.M1, IC9.M2, R1.2, R10.1, R2.1, R3.1, R4.1, R5.1, R6.1, R7.1, R8.1, R9.1, SV10.3, SV11.3, SV12.3, U$2.VCC
- new net N$80: IC6.STEP, U1.D21
- new net N$81: IC7.DIR, U1.D22
- new net N$82: IC7.STEP, U1.D23
- new net N$83: IC8.DIR, U1.D25
- new net N$84: IC8.STEP, U1.D26
- new net N$85: IC9.DIR, U1.D27
- new net N$86: IC9.STEP, U1.D32
- new net N$87: IC11A.Y2, U$5.+DCCONTROL
- new net N$88: IC10.STEP, U1.TX0
- new net N$89: IC11A.Y0, U$3.+DCCONTROL
- new net N$90: IC11A.Y1, U$4.+DCCONTROL
- new net N$91: SV10.1, U1.D35
- new net N$92: SV11.1, U1.D34
- new net N$93: IC10.DIR, U1.RX0
- new net N$94: C1.+, R1.1, SL2.2, U1.VP
- new net N$95: IC11A.A, U1.RX2
- new net N$96: IC11A.B, U1.TX2
- new net N$97: SV12.1, U1.VN
- net N$1: now also IC2.DIR, U1.D2; no longer IC2.GND1, IC3.GND1, IC4.GND1, IC5.GND1, IC6.GND1, IC7.GND1, IC8.GND1, IC9.GND1, U$1.GND
- net N$43: now also C1.-, IC1.GND, IC10.GND1, IC10.GND2, IC2.GND1, IC2.GND2, IC3.GND1, IC3.GND2, IC4.GND1, IC4.GND2, IC5.GND1, IC5.GND2, IC6.GND1, IC6.GND2, IC7.GND1, IC7.GND2, IC8.GND1, IC8.GND2, IC9.GND1, IC9.GND2, SL1.2, SL2.1, SV10.2, SV11.2, SV12.2, U$2.GND, U$3.-DCCONTROL, U$4.-DCCONTROL, U$5.-DCCONTROL, U1.GND; no longer IC1.VO, R1.2, SV10.3, SV11.3, SV12.3, U$2.VCC
Other:
- note removed: "MOBILE PLATFORM STEPPER DRIVERS."
- note removed: "ROBOTIC ARM STEPPER DRIVERS."
- moved on the sheet: C1, F1, IC6, R1, SL1, SL2, SV1, SV10, SV11, SV12, SV13, SV19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
